File: braids_v50.kicad_pcb (KiCad board)
At the start: 2 copper layers, 78.7 x 106.7 mm, 120 parts, among them IC1 74HC595D, IC10 TL072, IC2 74HC595D, IC3 LM4040B25, IC4 MCP3204, IC5 DAC8551, IC6 LM1117-3.3, IC7 MCP6004, IC8 LM4040B10, IC9 TL074D, J1 PJ301_THONKICONN6, J2 PJ301_THONKICONN6, J3 PJ301_THONKICONN6, J4 PJ301_THONKICONN6, J5 PJ301_THONKICONN6, J6 PJ301_THONKICONN6, Q1 MMBT3904, Q2 MMBT3904, Q3 MMBT3904, Q4 MMBT3904, Q5 8MHz, Q6 MMBT3904, SW1 EC12E_SW

Commit message: Clean up incorrectly converted vias in prep to re-lay them
Other:
- board text removed: "FillOverPAD:GND:10:455"
- board text removed: "FillOverPAD:GND:110:455"
- board text removed: "FillOverPAD:GND:115:455"
- board text removed: "FillOverPAD:GND:126:455"
- board text removed: "FillOverPAD:GND:12:455"
- board text removed: "FillOverPAD:GND:131:455"
- board text removed: "FillOverPAD:GND:136:455"
- board text removed: "FillOverPAD:GND:144:455"
- board text removed: "FillOverPAD:GND:149:455"
- board text removed: "FillOverPAD:GND:14:455"
- board text removed: "FillOverPAD:GND:159:455"
- board text removed: "FillOverPAD:GND:160:455"
- board text removed: "FillOverPAD:GND:165:455"
- board text removed: "FillOverPAD:GND:167:455"
- board text removed: "FillOverPAD:GND:16:455"
- board text removed: "FillOverPAD:GND:172:455"
- board text removed: "FillOverPAD:GND:173:455"
- board text removed: "FillOverPAD:GND:174:455"
- board text removed: "FillOverPAD:GND:177:455"
- board text removed: "FillOverPAD:GND:17:455"
- board text removed: "FillOverPAD:GND:182:455"
- board text removed: "FillOverPAD:GND:184:455"
- board text removed: "FillOverPAD:GND:189:455"
- board text removed: "FillOverPAD:GND:191:455"
- board text removed: "FillOverPAD:GND:196:455"
- board text removed: "FillOverPAD:GND:19:455"
- board text removed: "FillOverPAD:GND:22:455"
- board text removed: "FillOverPAD:GND:248:455"
- board text removed: "FillOverPAD:GND:24:455"
- board text removed: "FillOverPAD:GND:251:455"
- board text removed: "FillOverPAD:GND:254:455"
- board text removed: "FillOverPAD:GND:257:455"
- board text removed: "FillOverPAD:GND:262:455"
- board text removed: "FillOverPAD:GND:2:455"
- board text removed: "FillOverPAD:GND:30:455"
- board text removed: "FillOverPAD:GND:336:455"
- board text removed: "FillOverPAD:GND:36:455"
- board text removed: "FillOverPAD:GND:38:455"
- board text removed: "FillOverPAD:GND:39:455"
- board text removed: "FillOverPAD:GND:400:455"
- board text removed: "FillOverPAD:GND:401:455"
- board text removed: "FillOverPAD:GND:415:455"
- board text removed: "FillOverPAD:GND:427:455"
- board text removed: "FillOverPAD:GND:430:455"
- board text removed: "FillOverPAD:GND:442:455"
- board text removed: "FillOverPAD:GND:44:455"
- board text removed: "FillOverPAD:GND:453:455"
- board text removed: "FillOverPAD:GND:454:455"
- board text removed: "FillOverPAD:GND:46:455"
- board text removed: "FillOverPAD:GND:4:455"
- board text removed: "FillOverPAD:GND:50:455"
- board text removed: "FillOverPAD:GND:52:455"
- board text removed: "FillOverPAD:GND:53:455"
- board text removed: "FillOverPAD:GND:56:455"
- board text removed: "FillOverPAD:GND:59:455"
- board text removed: "FillOverPAD:GND:62:455"
- board text removed: "FillOverPAD:GND:6:455"
- board text removed: "FillOverPAD:GND:8:455"
- board text removed: "V:GND:100:108"
- board text removed: "V:GND:101:108"
- board text removed: "V:GND:102:108"
- board text removed: "V:GND:103:108"
- board text removed: "V:GND:104:108"
- board text removed: "V:GND:105:108"
- board text removed: "V:GND:106:108"
- board text removed: "V:GND:107:108"
- board text removed: "V:GND:108:108"
- board text removed: "V:GND:10:108"
- board text removed: "V:GND:11:108"
- board text removed: "V:GND:12:108"
- board text removed: "V:GND:13:108"
- board text removed: "V:GND:14:108"
- board text removed: "V:GND:15:108"
- board text removed: "V:GND:16:108"
- board text removed: "V:GND:17:108"
- board text removed: "V:GND:18:108"
- board text removed: "V:GND:19:108"
- board text removed: "V:GND:1:108"
- board text removed: "V:GND:20:108"
- board text removed: "V:GND:21:108"
- board text removed: "V:GND:22:108"
- board text removed: "V:GND:23:108"
- board text removed: "V:GND:24:108"
- board text removed: "V:GND:25:108"
- board text removed: "V:GND:26:108"
- board text removed: "V:GND:27:108"
- board text removed: "V:GND:28:108"
- board text removed: "V:GND:29:108"
- board text removed: "V:GND:2:108"
- board text removed: "V:GND:30:108"
- board text removed: "V:GND:31:108"
- board text removed: "V:GND:32:108"
- board text removed: "V:GND:33:108"
- board text removed: "V:GND:34:108"
- board text removed: "V:GND:35:108"
- board text removed: "V:GND:36:108"
- board text removed: "V:GND:37:108"
- board text removed: "V:GND:38:108"
- board text removed: "V:GND:39:108"
- board text removed: "V:GND:3:108"
- board text removed: "V:GND:40:108"
- board text removed: "V:GND:41:108"
- board text removed: "V:GND:42:108"
- board text removed: "V:GND:43:108"
- board text removed: "V:GND:44:108"
- board text removed: "V:GND:45:108"
- board text removed: "V:GND:46:108"
- board text removed: "V:GND:47:108"
- board text removed: "V:GND:48:108"
- board text removed: "V:GND:49:108"
- board text removed: "V:GND:4:108"
- board text removed: "V:GND:50:108"
- board text removed: "V:GND:51:108"
- board text removed: "V:GND:52:108"
- board text removed: "V:GND:53:108"
- board text removed: "V:GND:54:108"
- board text removed: "V:GND:55:108"
- board text removed: "V:GND:56:108"
- board text removed: "V:GND:57:108"
- board text removed: "V:GND:58:108"
- board text removed: "V:GND:59:108"
- board text removed: "V:GND:5:108"
- board text removed: "V:GND:60:108"
- board text removed: "V:GND:61:108"
- board text removed: "V:GND:62:108"
- board text removed: "V:GND:63:108"
- board text removed: "V:GND:64:108"
- board text removed: "V:GND:65:108"
- board text removed: "V:GND:66:108"
- board text removed: "V:GND:67:108"
- board text removed: "V:GND:68:108"
- board text removed: "V:GND:69:108"
- board text removed: "V:GND:6:108"
- board text removed: "V:GND:70:108"
- board text removed: "V:GND:71:108"
- board text removed: "V:GND:72:108"
- board text removed: "V:GND:73:108"
- board text removed: "V:GND:74:108"
- board text removed: "V:GND:75:108"
- board text removed: "V:GND:76:108"
- board text removed: "V:GND:77:108"
- board text removed: "V:GND:78:108"
- board text removed: "V:GND:79:108"
- board text removed: "V:GND:7:108"
- board text removed: "V:GND:80:108"
- board text removed: "V:GND:81:108"
- board text removed: "V:GND:82:108"
- board text removed: "V:GND:83:108"
- board text removed: "V:GND:84:108"
- board text removed: "V:GND:85:108"
- board text removed: "V:GND:86:108"
- board text removed: "V:GND:87:108"
- board text removed: "V:GND:88:108"
- board text removed: "V:GND:89:108"
- board text removed: "V:GND:8:108"
- board text removed: "V:GND:90:108"
- board text removed: "V:GND:91:108"
- board text removed: "V:GND:92:108"
- board text removed: "V:GND:93:108"
- board text removed: "V:GND:94:108"
- board text removed: "V:GND:95:108"
- board text removed: "V:GND:96:108"
- board text removed: "V:GND:97:108"
- board text removed: "V:GND:98:108"
- board text removed: "V:GND:99:108"
- board text removed: "V:GND:9:108"
